File: Lifedatalink_v1_revA.kicad_pcb (KiCad board)
At the start: 4 copper layers, 53.7 x 68.8 mm, 69 parts, among them J1 DX07S024XJ1R1100, J2 5015680207, J3 Conn_01x06, J4 Conn_01x02, J5 Conn_01x06, J6 Conn_01x06, J7 ECG_IN, M1 MLX90614ESF-AAA-000-TU, Q1 CSD23280F3, SW1 SW_Push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

Commit message: Replace the BLE module with an ISP1807-LR-RS
Parts:
- removed C1: 12pF, Capacitor_SMD:C_0402_1005Metric
- removed C2: 10pF, Capacitor_SMD:C_0402_1005Metric
- removed Y1: Crystal, ABS05-32.768KHZ-T:ABS05-32.768KHZ-T
- U1: value NORA-B106-00B -> ISP1807-LR-RS; footprint Footprints:XCVR_NORA-B106-00B -> Footprints:ISP1807-LR-RS
- moved U1 3.42 mm to (148.4, 125.0), turned to 0 degrees
Connections:
- net /NORA_I2S_SD_EXT renamed /ISP_I2S_SD_EXT
- A1 pad 15: /NORA_UART_RX -> /ISP_UART_RX
- A1 pad 16: /NORA_UART_TX -> /ISP_UART_TX
- J1 pad A6: /NORA_USB_DP -> /ISP_USB_DP
- J1 pad A7: /NORA_USB_DM -> /ISP_USB_DM
- J1 pad B6: /NORA_USB_DP -> /ISP_USB_DP
- J1 pad B7: /NORA_USB_DM -> /ISP_USB_DM
- J4 pad 1: /NORA_SWDCLK -> /ISP_SWDCLK
- J4 pad 2: /NORA_SWDIO -> /ISP_SWDIO
- J5 pad 1: /NORA_I2C_SCL -> /ISP_I2C_SCL
- J5 pad 2: /NORA_I2C_SDA -> /ISP_I2C_SDA
- J5 pad 3: /NORA_I2S_WS -> /ISP_I2S_WS
- J5 pad 4: /NORA_I2S_SCK -> /ISP_I2S_SCK
- J5 pad 5: /NORA_I2S_SD -> /ISP_I2S_SD
- MICL1 pad 1: /NORA_I2S_WS_EXT -> /ISP_I2S_WS
- MICL1 pad 4: /NORA_I2S_SCK_EXT -> /ISP_I2S_SCK
- MICR1 pad 1: /NORA_I2S_WS_EXT -> /ISP_I2S_WS
- MICR1 pad 4: /NORA_I2S_SCK_EXT -> /ISP_I2S_SCK
- R18 pad 1: ECG_N -> ECG_P
- SW1 pad 1: Net-(U1-P1.12) -> Net-(U1-P0_08)
- U10 pad 3: /NORA_USB_DP -> /ISP_USB_DP
- U10 pad 5: /NORA_USB_DM -> /ISP_USB_DM
- U6 pad 8: /NORA_I2C_SDA -> /ISP_I2C_SDA
- U6 pad 9: /NORA_I2C_SCL -> /ISP_I2C_SCL
- U8 pad 4: /NORA_I2C_SCL -> /ISP_I2C_SCL
- U8 pad 6: /NORA_I2C_SDA -> /ISP_I2C_SDA
