File: Lifedatalink_v1_revA.kicad_sch (KiCad schematic)
At the start: 69 parts, among them J1 DX07S024XJ1R1100, J2 5015680207, J3 Conn_01x06, J4 Conn_01x02, J5 Conn_01x06, J6 Conn_01x06, J7 ECG_IN, M1 MLX90614ESF-AAA-000-TU, Q1 CSD23280F3, SW1 SW_Push, U1 NORA-B106-00B, U10 TPD2E001IDRLRQ1, U2 TCR3UG33A,LF, U3 ADS1293CISQE/NOPB, U4 MCP73831T-3ACI{slash}MC, U5 LMT70AYFQT, U6 MAX86150EFF+T, U7 TCR3UG18A,LF, U8 LIS331DLHTR, U9 LTST-E263CEGBK, Y1 Crystal, Y2 Crystal

Commit message: Replace the BLE module with a BL5340 (453-00053R)
Parts:
- removed U1: NORA-B106-00B, Footprints:XCVR_NORA-B106-00B, symbol NORA-B106-00B:NORA-B106-00B
- added U1: 453-00052R, Footprints:45300052R, symbol 453-00052R:453-00052R
Connections:
- net +3V3: now also U1.31 (VDD), U1.35 (VDD_HV)
- net +5V: now also U1.40 (VBUS)
- net ACCEL_CS: now also U1.3 (P0.24)
- net ACCEL_INT1: now also U1.4 (P0.27/AIN6)
- net ACCEL_INT2: now also U1.5 (P1.09)
- net ADS_ALARMB: now also U1.15 (P0.19)
- net ADS_CLK: now also U1.9 (P1.06)
- net ADS_CSB: now also U1.14 (P0.20)
- net ADS_DRDYB: now also U1.10 (P1.05)
- net ADS_SCLK: now also U1.13 (P1.04)
- net ADS_SDI: now also U1.12 (P0.22)
- net ADS_SDO: now also U1.11 (P0.21)
- net BAT_VDIV: now also U1.63 (P0.04_/_AIN0)
- net GND: now also U1.1 (GND_1), U1.19 (GND_2), U1.21 (GND_3), U1.29 (GND_4), U1.30 (GND_5), U1.33 (GND_6), U1.39 (GND_7), U1.44 (GND_8), U1.59 (GND_9), U1.66 (GND_10), U1.67 (GND_11), U1.68 (GND_12), U1.69 (GND_13), U1.70 (GND_14), U1.71 (GND_15), U1.73 (GND_16), U1.74 (GND_17), U1.75 (GND_18)
- net LED_DATA: now also U1.52 (P0.30)
- net MCP73831_STAT: now also U1.2 (P0.26_/_AIN5)
- net ~{MAX_INT}: now also U1.8 (P1.07)
- net at C2.1, Y1.2: now also U1.34 (P0.00_/_XL1)
- net at C1.1, Y1.1: now also U1.32 (P0.01_/_XL2)
- net at SW1.1: now also U1.58 (P0.29)
- net NORA_I2C_SCL renamed ISP_I2C_SCL
- net ISP_I2C_SCL: now also U1.47 (P1.13)
- net NORA_I2C_SDA renamed ISP_I2C_SDA
- net ISP_I2C_SDA: now also U1.48 (P1.14)
- net NORA_I2S_SCK renamed ISP_I2S_SCK
- net ISP_I2S_SCK: now also U1.50 (P1.11)
- net NORA_I2S_SD renamed ISP_I2S_SD
- net ISP_I2S_SD: now also U1.51 (P0.31)
- net NORA_I2S_SD_EXT renamed ISP_I2S_SD_EXT
- net NORA_I2S_WS renamed ISP_I2S_WS
- net ISP_I2S_WS: now also U1.49 (P1.12)
- net NORA_SWDCLK renamed ISP_SWDCLK
- net ISP_SWDCLK: now also U1.56 (SWDCLK)
- net NORA_SWDIO renamed ISP_SWDIO
- net ISP_SWDIO: now also U1.55 (SWDIO)
- net NORA_UART_RX renamed ISP_UART_RX
- net ISP_UART_RX: now also U1.7 (P1.08)
- net NORA_UART_TX renamed ISP_UART_TX
- net ISP_UART_TX: now also U1.6 (P0.25_/_AIN4)
- net NORA_USB_DM renamed ISP_USB_DM
- net ISP_USB_DM: now also U1.42 (D-)
- net NORA_USB_DP renamed ISP_USB_DP
- net ISP_USB_DP: now also U1.36 (D+)
Other:
- moved on the sheet: A1, C1, C2, J4, R1, R2, SW1, U9, Y1
